File: powerBoard_v1/powerBoard.brd (EAGLE design)
At the start: 81.3 x 58.1 mm, 43 parts, among them IC1 7805T, IC2 317T, IC3 317T, IC4 317T, IC5 7808T, J1 DCJ0202

Commit message: powerBoard schematic corrected
Parts:
- removed SL1, SL10, SL11, SL12, SL13, SL14, SL15, SL16, SL17, SL18, SL2, SL3, SL4, SL5, SL6, SL7, SL8, SL9: (no value), con-amp-quick:02P
- added X1, X10, X11, X12, X13, X14, X15, X16, X17, X18, X2, X3, X4, X5, X6, X7, X8, X9: (no value), con-ptr500:AK300/2
- R12: device pot:CA6V -> pot:RJ9W
- moved R5 11.4 mm to (54.6, 33.0)
- moved R6 11.4 mm to (54.6, 35.6)
- moved IC1 11.4 mm to (71.1, 26.7)
- moved IC5 11.4 mm to (35.6, 26.7)
- moved C1 11.4 mm to (17.8, 34.3)
- moved C3 11.4 mm to (54.6, 50.8)
- moved C4 11.4 mm to (5.08, 54.6)
- moved C5 11.4 mm to (25.4, 57.1)
- moved IC2 11.4 mm to (67.3, 45.7)
- moved IC3 11.4 mm to (7.62, 36.8)
- moved IC4 11.4 mm to (34.3, 43.2)
- moved R1 11.4 mm to (54.6, 45.7)
- moved R10 11.4 mm to (24.1, 44.5)
- moved R11 11.4 mm to (41.9, 50.8)
- moved R13 11.4 mm to (44.5, 50.8)
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Connections:
- net +12V: now also X1.1, X2.1, X3.1; no longer SL1.1, SL2.1, SL3.1
- net +3V3: now also X10.1, X11.1, X12.1; no longer SL16.1, SL17.1, SL18.1
- net +5V: now also X7.1, X8.1, X9.1; no longer SL7.1, SL8.1, SL9.1
- net GND: now also X1.2, X10.2, X11.2, X12.2, X13.2, X14.2, X15.2, X16.2, X17.2, X18.2, X2.2, X3.2, X4.2, X5.2, X6.2, X7.2, X8.2, X9.2; no longer SL1.2, SL10.2, SL11.2, SL12.2, SL13.2, SL14.2, SL15.2, SL16.2, SL17.2, SL18.2, SL2.2, SL3.2, SL4.2, SL5.2, SL6.2, SL7.2, SL8.2, SL9.2
- net VCC: now also X13.1, X14.1, X15.1; no longer SL10.1, SL11.1, SL12.1
- net VCC/2: now also X16.1, X17.1, X18.1; no longer SL13.1, SL14.1, SL15.1
- net VDD: now also X4.1, X5.1, X6.1; no longer SL4.1, SL5.1, SL6.1
Routing:
- net GND: track 402.6 -> 0.00 mm
- net +12V: track 163.8 -> 0.00 mm
- net VCC: track 104.8 -> 0.00 mm
- net +3V3: track 70.4 -> 0.00 mm
- net VCC/2: track 39.9 -> 0.00 mm
- net +5V: track 35.3 -> 0.00 mm
- net VDD: track 33.5 -> 0.00 mm
- net N$2: track 30.5 -> 0.00 mm
- net N$12: track 23.7 -> 0.00 mm
- net N$9: track 18.8 -> 0.00 mm
- net N$4: track 16.5 -> 0.00 mm
- net N$5: track 5.08 -> 0.00 mm
- net N$13: track 2.54 -> 0.00 mm
- net N$7: track 2.54 -> 0.00 mm
- net N$6: track 2.54 -> 0.00 mm

Commit message: board completed
Parts:
- moved X10 219.2 mm to (148.6, 52.1), turned to 180 degrees
- moved X18 216.9 mm to (21.6, 52.1), turned to 180 degrees
- moved X16 210.6 mm to (52.1, 52.1), turned to 180 degrees
- moved X13 206.9 mm to (100.3, 52.1), turned to 180 degrees
- moved X12 206.6 mm to (118.1, 52.1), turned to 180 degrees
- moved X15 203.5 mm to (69.8, 52.1), turned to 180 degrees
- moved X17 201.8 mm to (36.8, 52.1), turned to 180 degrees
- moved X11 198.2 mm to (133.3, 52.1), turned to 180 degrees
- moved X14 191.3 mm to (85.1, 52.1), turned to 180 degrees
- moved X9 189.7 mm to (148.6, 6.35)
- moved X8 159.0 mm to (133.3, 6.35)
- moved X7 155.4 mm to (118.1, 6.35)
- moved X6 133.7 mm to (100.3, 6.35)
- moved X5 104.2 mm to (85.1, 6.35)
- moved X4 100.4 mm to (69.8, 6.35)
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Routing:
- net GND: track 0.00 -> 650.6 mm
- net +12V: track 0.00 -> 226.1 mm
- net VCC: track 0.00 -> 110.3 mm
- net +3V3: track 0.00 -> 100.5 mm
- net VCC/2: track 0.00 -> 84.4 mm
- net VDD: track 0.00 -> 64.1 mm
- net +5V: track 0.00 -> 64.1 mm
- net N$4: track 0.00 -> 33.1 mm
- net N$2: track 0.00 -> 19.4 mm
- net N$12: track 0.00 -> 15.7 mm
- net N$5: track 0.00 -> 13.2 mm
- net N$13: track 0.00 -> 9.94 mm
- net N$9: track 0.00 -> 6.35 mm
- net N$7: track 0.00 -> 3.81 mm
- net N$6: track 0.00 -> 3.81 mm
Other:
- board size 81.3 x 58.1 mm -> 158.7 x 58.1 mm
- board text added: "powerBoard_v1"
- board text removed: "powerBoard v1"
